File: io_board/CM5IO.kicad_sch (KiCad schematic)
At the start: 12 parts, among them J11 USB_C_Receptacle_USB2.0

Commit message: Cleaned up schematic
Parts:
- removed H1, H2, H3, H4, H5, H6, H7, H8: MountingHole, CM5IO:MountingHole_2.7mm_M2.5_DIN965, symbol Mechanical:MountingHole
Connections:
- no-connect marks 2 -> 12
Other:
- removed sheet PCIe-M2
- added sheet CM5_ExtraIO (CM5_Extra_IO.kicad_sch)
- note added: "Connectors ------- CSI/DSI 0 CSI/DSI 1"
- note added: "Connectors ------- Ethernet SDCARD 40way RPI Jumpers Fan"
- note added: "Connectors ------- USB 3 Serial I2C SPI GPIO"
- note removed: "Connectors ------ M2 MKey"
- note removed: "Connectors ------- Ethernet SDCARD 40way RPI Jumpers Fan Battery"
- note removed: "Connectors ------- HDMI 0 HDMI 1 CSI/DSI 0 CSI/DSI 1"
