File: io_board/CM5_HighSpeed.kicad_sch (KiCad schematic)
At the start: 19 parts, among them J10 690-019-298-412, J12 USB3_A, J16 Conn_01x22_Female, J22 690-019-298-412, J5 Conn_01x22_Female, J6 THD-02-R, U12 RT9742SNGV, U6 AP22653W6

Commit message: Cleaned up schematic
Parts:
- removed C12, C13: 100n, Capacitor_SMD:C_0402_1005Metric, symbol Device:C
- removed J10, J22: 690-019-298-412, CM5IO:EDAC 690-019-298-412, symbol CM5IO:HDMI_A_1.4
- removed J12: USB3_A, CM5IO:MTCONN_UBAF30-D2011, symbol CM5IO:USB3_A
- removed J6: THD-02-R, Connector_PinHeader_2.54mm:PinHeader_2x02_P2.54mm_Vertical, symbol Connector_Generic:Conn_02x02_Odd_Even
- removed R6, R7: 2.2K 1%, Resistor_SMD:R_0402_1005Metric, symbol Device:R
- removed U12: RT9742SNGV, Package_TO_SOT_SMD:TSOT-23_HandSoldering, symbol CM5IO:RT9742SNGV
Connections:
- no-connect marks 4 -> 2
Other:
- note added: "CSI Connectors"
- note removed: "DSI/CSI Connectors"
- note removed: "Jumpers to be fitted if DPHY1 is used"
- note removed: "Stacked USB connectors"
- note removed: "USB 3 Pairs P/N swapped to help routing"
